Commit message: Updated a1.py to include working visualization

File: systems/A1/A1_description/urdf/a1_foot_collision.urdf (robot description, URDF)
Before this commit: robot a1_description, 19 links, 18 joints
Links:
- link FL_calf: geometry visual mesh filename=../meshes/calf.obj scale=1 1 1
- link FL_hip: geometry visual mesh filename=../meshes/hip.obj scale=1 1 1
- link FL_thigh: geometry visual mesh filename=../meshes/thigh.obj scale=1 1 1
- link FR_calf: geometry visual mesh filename=../meshes/calf.obj scale=1 1 1
- link FR_hip: geometry visual mesh filename=../meshes/hip.obj scale=1 1 1
- link FR_thigh: geometry visual mesh filename=../meshes/thigh_mirror.obj scale=1 1 1
- link RL_calf: geometry visual mesh filename=../meshes/calf.obj scale=1 1 1
- link RL_hip: geometry visual mesh filename=../meshes/hip.obj scale=1 1 1
- link RL_thigh: geometry visual mesh filename=../meshes/thigh.obj scale=1 1 1
- link RR_calf: geometry visual mesh filename=../meshes/calf.obj scale=1 1 1
- link RR_hip: geometry visual mesh filename=../meshes/hip.obj scale=1 1 1
- link RR_thigh: geometry visual mesh filename=../meshes/thigh_mirror.obj scale=1 1 1
- link trunk: geometry visual mesh filename=../meshes/trunk.obj scale=1 1 1
